File: intraoral_led_driver.sch (KiCad schematic (older format))
At the start: 32 parts, among them J1 CONN_01X04, J2 CONN_01X03, J3 CONN_01X04, J4 CONN_01X02, J5 CONN_01X02, Q1 Si2318DS-T1, Q2 Si2318DS-T1, SW1 SW_SPST, U1 LT3478-1, U3 AD5247

Commit message: update for new connector
Parts:
- J1, J3: symbol CONN_01X04 -> Conn_01x04
- J2: symbol CONN_01X03 -> Conn_01x03
- J4, J5: symbol CONN_01X02 -> Conn_01x02
Changed lines of the file:
@@
 EESchema Schematic File Version 2
+LIBS:intraoral_led_driver-rescue
 LIBS:power
 LIBS:device
@@
 LIBS:sensors
 LIBS:switches
+LIBS:custom_library
 LIBS:fiducial
-LIBS:custom_library
 LIBS:intraoral_led_driver-cache
 EELAYER 25 0
@@
 V_w+
 $Comp
-L CONN_01X04 J3
+L Conn_01x04 J3
 U 1 1 59360C25
-P 13250 5305
-F 0 "J3" H 13250 5555 50  0000 C CNN
-F 1 "CONN_01X04" V 13350 5305 50  0000 C CNN
-F 2 "Connectors_JST:JST_PH_S4B-PH-SM4-TB_04x2.00mm_Angled" H 13250 5305 50  0001 C CNN
-F 3 "" H 13250 5305 50  0001 C CNN
-	1    13250 5305
+P 13250 5355
+F 0 "J3" H 13250 5605 50  0000 C CNN
+F 1 "CONN_01X04" V 13350 5355 50  0000 C CNN
+F 2 "Connectors_JST:JST_PH_S4B-PH-SM4-TB_04x2.00mm_Angled" H 13250 5355 50  0001 C CNN
+F 3 "" H 13250 5355 50  0001 C CNN
+	1    13250 5355
 	1    0    0    1
 $EndComp
 $Comp
-L CONN_01X04 J1
+L Conn_01x04 J1
 U 1 1 59362528
-P 6475 7645
-F 0 "J1" H 6475 7895 50  0000 C CNN
-F 1 "CONN_01X04" V 6575 7645 50  0000 C CNN
-F 2 "Connectors_JST:JST_PH_S4B-PH-SM4-TB_04x2.00mm_Angled" H 6475 7645 50  0001 C CNN
-F 3 "" H 6475 7645 50  0001 C CNN
-	1    6475 7645
+P 6425 7645
+F 0 "J1" H 6425 7895 50  0000 C CNN
+F 1 "CONN_01X04" V 6525 7645 50  0000 C CNN
+F 2 "Connectors_JST:JST_PH_S4B-PH-SM4-TB_04x2.00mm_Angled" H 6425 7645 50  0001 C CNN
+F 3 "" H 6425 7645 50  0001 C CNN
+	1    6425 7645
 	0    -1   1    0
 $EndComp
 $Comp
-L CONN_01X03 J2
+L Conn_01x03 J2
 U 1 1 5936182A
 P 9755 8155
@@
 	9755 7835 9755 7955
 $Comp
-L CONN_01X02 J5
+L Conn_01x02 J5
 U 1 1 5936502E
-P 3920 3545
-F 0 "J5" H 3920 3695 50  0000 C CNN
-F 1 "CONN_01X02" V 4020 3545 50  0000 C CNN
-F 2 "Connectors_JST:JST_PH_S2B-PH-SM4-TB_02x2.00mm_Angled" H 3920 3545 50  0001 C CNN
-F 3 "" H 3920 3545 50  0001 C CNN
-	1    3920 3545
+P 3870 3545
+F 0 "J5" H 3870 3695 50  0000 C CNN
+F 1 "CONN_01X02" V 3970 3545 50  0000 C CNN
+F 2 "Connectors_JST:JST_PH_S2B-PH-SM4-TB_02x2.00mm_Angled" H 3870 3545 50  0001 C CNN
+F 3 "" H 3870 3545 50  0001 C CNN
+	1    3870 3545
 	0    -1   -1   0
 $EndComp
 $Comp
-L CONN_01X02 J4
+L Conn_01x02 J4
 U 1 1 593650F2
-P 2430 4985
-F 0 "J4" H 2430 5135 50  0000 C CNN
-F 1 "CONN_01X02" V 2530 4985 50  0000 C CNN
-F 2 "Connectors_JST:JST_PH_S2B-PH-SM4-TB_02x2.00mm_Angled" H 2430 4985 50  0001 C CNN
-F 3 "" H 2430 4985 50  0001 C CNN
-	1    2430 4985
+P 2430 5035
+F 0 "J4" H 2430 5185 50  0000 C CNN
+F 1 "CONN_01X02" V 2530 5035 50  0000 C CNN
+F 2 "Connectors_JST:JST_PH_S2B-PH-SM4-TB_02x2.00mm_Angled" H 2430 5035 50  0001 C CNN
+F 3 "" H 2430 5035 50  0001 C CNN
+	1    2430 5035
 	-1   0    0    1
 $EndComp
